File: v1.2/PCB/circuitdraft.brd (EAGLE design)
At the start: 31.2 x 35.4 mm, 23 parts, among them Y1 CY16BPS

Commit message: Added switch. Passes DRC
Final 1.2
Parts:
- added BAT, PWRSW: (no value), pinhead:1X02
- moved RPROG 4.10 mm to (13.2, 21.2), turned to 270 degrees
Connections:
- new net BATCHARGE: BAT.1, CHRG.3, COUT.1, PWRSW.2
- net GND: now also BAT.2
- net VBAT: now also PWRSW.1; no longer CHRG.3, COUT.1
Routing:
- net BATCHARGE: track 0.00 -> 18.3 mm, vias 0 -> 1
- net VBAT: track 12.8 -> 17.6 mm
Changed lines of the file:
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@@
 <wire x1="43" y1="38.4" x2="11.8" y2="38.4" width="0" layer="20"/>
 <wire x1="11.8" y1="38.4" x2="11.8" y2="3" width="0" layer="20"/>
-<text x="14.5" y="14.6" size="1.778" layer="22" rot="MR180">MU3DPC Hand v1.2</text>
+<text x="21.7" y="14.2" size="1.778" layer="22" rot="MR180">MU3DPC Hand v1.2</text>
 <dimension x1="11.8" y1="3" x2="43" y2="3" x3="27.4" y3="0.5" textsize="1.778" layer="1"/>
 <dimension x1="43" y1="3" x2="43" y2="38.4" x3="48.1" y3="20.7" textsize="1.778" layer="1"/>
@@
 <attribute name="SPICEPREFIX" value="C" x="20.2" y="23.2" size="1.778" layer="27" rot="R90" display="off"/>
 </element>
-<element name="RPROG" library="3DPC" package="R0603" package3d_urn="urn:adsk.eagle:package:23555/3" value="2 kOhm" x="16.2" y="18.4" smashed="yes" rot="R180">
-<attribute name="NAME" x="21.035" y="16.865" size="1.27" layer="25" rot="R180"/>
-<attribute name="POPULARITY" value="77" x="16.2" y="18.4" size="1.778" layer="27" rot="R180" display="off"/>
-<attribute name="SPICEPREFIX" value="R" x="16.2" y="18.4" size="1.778" layer="27" rot="R180" display="off"/>
+<element name="RPROG" library="3DPC" package="R0603" package3d_urn="urn:adsk.eagle:package:23555/3" value="2 kOhm" x="13.2" y="21.2" smashed="yes" rot="R270">
+<attribute name="NAME" x="14.735" y="26.035" size="1.27" layer="25" rot="R270"/>
+<attribute name="POPULARITY" value="77" x="13.2" y="21.2" size="1.778" layer="27" rot="R270" display="off"/>
+<attribute name="SPICEPREFIX" value="R" x="13.2" y="21.2" size="1.778" layer="27" rot="R270" display="off"/>
 </element>
 <element name="SJ1" library="jumper" library_urn="urn:adsk.eagle:library:252" package="SJ" package3d_urn="urn:adsk.eagle:package:15471/1" value="" x="17.5" y="25.3" smashed="yes">
@@
 <attribute name="POPULARITY" value="33" x="17.5" y="25.3" size="1.778" layer="27" display="off"/>
 <attribute name="VALUE" x="17.9001" y="25.3" size="0.02" layer="27"/>
+</element>
+<element name="BAT" library="pinhead" library_urn="urn:adsk.eagle:library:325" package="1X02" package3d_urn="urn:adsk.eagle:package:22435/2" value="" x="17.4" y="16.5" smashed="yes" rot="R90">
+<attribute name="NAME" x="19.1288" y="17.4162" size="1.27" layer="25" ratio="10" rot="R270"/>
+<attribute name="POPULARITY" value="98" x="17.4" y="16.5" size="1.778" layer="27" rot="R90" display="off"/>
+<attribute name="VALUE" x="20.575" y="13.96" size="1.27" layer="27" rot="R90"/>
+</element>
+<element name="PWRSW" library="pinhead" library_urn="urn:adsk.eagle:library:325" package="1X02" package3d_urn="urn:adsk.eagle:package:22435/2" value="" x="14" y="16.5" smashed="yes" rot="R270">
+<attribute name="NAME" x="13.2838" y="12.1288" size="1.27" layer="25" ratio="10"/>
+<attribute name="POPULARITY" value="98" x="14" y="16.5" size="1.778" layer="27" rot="R270" display="off"/>
+<attribute name="VALUE" x="10.825" y="19.04" size="1.27" layer="27" rot="R270"/>
 </element>
 </elements>
@@
 <wire x1="24.3598" y1="16.8402" x2="23.6" y2="17.6" width="0.1524" layer="16"/>
 <via x="23.6" y="17.6" extent="1-16" drill="0.35"/>
-<wire x1="22.12" y1="17.66" x2="21.7986" y2="17.9814" width="0.1524" layer="1"/>
 <wire x1="17.1714" y1="20.3786" x2="15.4" y2="22.15" width="0.1524" layer="1"/>
 <wire x1="17.1714" y1="19.6782125" x2="17.1714" y2="20.3786" width="0.1524" layer="1"/>
-<wire x1="21.7986" y1="17.9814" x2="18.8682125" y2="17.9814" width="0.1524" layer="1"/>
-<wire x1="18.8682125" y1="17.9814" x2="17.1714" y2="19.6782125" width="0.1524" layer="1"/>
 <wire x1="22.12" y1="17.66" x2="23.54" y2="17.66" width="0.1524" layer="1"/>
 <wire x1="23.54" y1="17.66" x2="23.6" y2="17.6" width="0.1524" layer="1"/>
+<wire x1="18.572325" y1="18.7606" x2="18.0890125" y2="18.7606" width="0.1524" layer="1"/>
+<wire x1="18.0890125" y1="18.7606" x2="17.1714" y2="19.6782125" width="0.1524" layer="1"/>
+<wire x1="22.12" y1="17.66" x2="19.672925" y2="17.66" width="0.1524" layer="1"/>
+<wire x1="19.672925" y1="17.66" x2="18.572325" y2="18.7606" width="0.1524" layer="1"/>
 </signal>
 <signal name="MISO">
@@
 <via x="16.2" y="23.2" extent="1-16" drill="0.35"/>
 <via x="20" y="19.2" extent="1-16" drill="0.35"/>
+<contactref element="BAT" pad="2"/>
+<via x="19.5" y="9.8" extent="1-16" drill="0.35"/>
+<via x="29.8" y="10.9" extent="1-16" drill="0.35"/>
+<via x="29.6" y="18" extent="1-16" drill="0.35"/>
+<via x="30.6" y="15.9" extent="1-16" drill="0.35"/>
+<via x="25.8" y="20" extent="1-16" drill="0.35"/>
 </signal>
 <signal name="INTERRUPT">
@@
 <contactref element="IREG" pad="2"/>
 <wire x1="14" y1="31.03" x2="14" y2="28.49" width="1" layer="1"/>
-<contactref element="CHRG" pad="3"/>
-<contactref element="COUT" pad="1"/>
+<contactref element="PWRSW" pad="1"/>
 <contactref element="SJ1" pad="1"/>
-<wire x1="14" y1="28.49" x2="16.738" y2="25.752" width="1.016" layer="1"/>
-<wire x1="16.738" y1="25.752" x2="16.738" y2="25.3" width="1.016" layer="1"/>
-<wire x1="16.738" y1="25.3" x2="17.0174" y2="25.0206" width="1.016" layer="1"/>
-<wire x1="17.0174" y1="25.0206" x2="17.0174" y2="24.22635625" width="1.016" layer="1"/>
-<wire x1="18" y1="23.24375625" x2="18" y2="22.15" width="1.016" layer="1"/>
-<wire x1="17.0174" y1="24.22635625" x2="18" y2="23.24375625" width="1.016" layer="1"/>
-<wire x1="20.2" y1="22.35" x2="20" y2="22.15" width="1.016" layer="1"/>
-<wire x1="20" y1="22.15" x2="18" y2="22.15" width="1.016" layer="1"/>
+<wire x1="14" y1="28.49" x2="14" y2="17.77" width="1.016" layer="16"/>
+<wire x1="16.738" y1="25.3" x2="14" y2="28.038" width="1" layer="1"/>
+<wire x1="14" y1="28.038" x2="14" y2="28.49" width="1" layer="1"/>
 </signal>
 <signal name="N$1">
@@
 <contactref element="CHRG" pad="5"/>
 <contactref element="RPROG" pad="2"/>
-<wire x1="15.4" y1="20.25" x2="15.4" y2="18.45" width="0.1524" layer="1"/>
-<wire x1="15.4" y1="18.45" x2="15.35" y2="18.4" width="0.1524" layer="1"/>
+<wire x1="15.4" y1="20.25" x2="14.3" y2="20.25" width="0.1524" layer="1"/>
+<wire x1="14.3" y1="20.25" x2="14.184209375" y2="20.35" width="0.1524" layer="1"/>
+<wire x1="14.184209375" y1="20.35" x2="13.2" y2="20.35" width="0.1524" layer="1"/>
 </signal>
 <signal name="N$2">
@@
 <wire x1="21" y1="25.3" x2="22.4" y2="23.9" width="0.1524" layer="1"/>
 </signal>
+<signal name="BATCHARGE" class="1">
+<contactref element="CHRG" pad="3"/>
+<contactref element="COUT" pad="1"/>
+<contactref element="BAT" pad="1"/>
+<contactref element="PWRSW" pad="2"/>
+<wire x1="14" y1="15.23" x2="17.4" y2="15.23" width="1.016" layer="1"/>
+<via x="17.6" y="23.4" extent="1-16" drill="0.35"/>
+<wire x1="17.6" y1="23.4" x2="18" y2="23" width="1" layer="1"/>
+<wire x1="18" y1="23" x2="18" y2="22.15" width="1" layer="1"/>
+<wire x1="20.2" y1="22.35" x2="20" y2="22.15" width="1" layer="1"/>
+<wire x1="20" y1="22.15" x2="18" y2="22.15" width="1" layer="1"/>
+<wire x1="18.74786875" y1="16.3556" x2="18.5256" y2="16.3556" width="1" layer="16"/>
+<wire x1="18.5256" y1="16.3556" x2="17.4" y2="15.23" width="1" layer="16"/>
+<wire x1="17.6" y1="23.4" x2="17.6" y2="22.94973125" width="1" layer="16"/>
+<wire x1="17.6" y1="22.94973125" x2="20.9544" y2="19.59533125" width="1" layer="16"/>
+<wire x1="20.9544" y1="19.59533125" x2="20.9544" y2="18.56213125" width="1" layer="16"/>
+<wire x1="20.9544" y1="18.56213125" x2="18.74786875" y2="16.3556" width="1" layer="16"/>
+</signal>
 </signals>
