File: v2.0/PCB/Hand v2.0.kicad_pcb (KiCad board)
At the start: 2 copper layers, 39 x 58 mm, 35 parts, among them J1 Conn_ARM_JTAG_SWD_10, M1 Index_Servo, M2 Middle_Servo, M3 Ring_Servo, M4 Pinky_Servo, M5 Thumb_Servo, SW1 Power_Switch

Commit message: v2.0 added version silkscreen and renamed files
Other:
- board text added: "MU3DPC Hand v2.0"
Changed lines of the file:
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@@
   (general
     (thickness 1.6)
-    (drawings 8)
+    (drawings 9)
     (tracks 217)
     (zones 0)
@@
     )
   )
+  (gr_text "MU3DPC Hand v2.0" (at 122.2 73.9) (layer F.SilkS)
+    (effects (font (size 1 1) (thickness 0.15)))
+  )
   (gr_line (start 152 72) (end 152 20) (layer Edge.Cuts) (width 0.05))
   (gr_line (start 116 75) (end 149 75) (layer Edge.Cuts) (width 0.05))
@@
   (segment (start 132.76499 39.38501) (end 132.76499 38.424994) (width 1.37) (layer F.Cu) (net 1) (status 1000000))
   (segment (start 131.95 41) (end 131.95 40.2) (width 1.37) (layer F.Cu) (net 1) (status 1000000))
-  (via (at 134.5 39.2) (size 0.8) (drill 0.4) (layers F.Cu B.Cu) (net 4))
-  (via (at 130.5 39.2) (size 0.8) (drill 0.4) (layers F.Cu B.Cu) (net 4))
   (segment (start 125.05 34) (end 126 33.05) (width 0.25) (layer F.Cu) (net 2))
   (segment (start 122 34) (end 125.05 34) (width 0.25) (layer F.Cu) (net 2))
@@
   (segment (start 131.6 61) (end 130.525 61) (width 0.25) (layer B.Cu) (net 3))
   (segment (start 143 68) (end 131.213285 68) (width 0.25) (layer B.Cu) (net 3))
+  (via (at 134.5 39.2) (size 0.8) (drill 0.4) (layers F.Cu B.Cu) (net 4))
+  (via (at 130.5 39.2) (size 0.8) (drill 0.4) (layers F.Cu B.Cu) (net 4))
   (segment (start 122.5 41) (end 122 40.5) (width 0.25) (layer F.Cu) (net 4))
   (segment (start 125.95 41) (end 122.5 41) (width 0.25) (layer F.Cu) (net 4))

Commit message: began swapping arm chips
Parts:
- removed MCU1: ATSAMD11C14A-SS, Package_SO:SOIC-14_3.9x8.7mm_P1.27mm
- removed R10: 1000ohm, Resistor_SMD:R_0805_2012Metric_Pad1.15x1.40mm_HandSolder
- added C10: 100nF, Capacitor_SMD:C_0805_2012Metric_Pad1.15x1.40mm_HandSolder, F.Cu at (102.8, 53.4)
- added C11: 4.7uF, Capacitor_SMD:C_0805_2012Metric_Pad1.15x1.40mm_HandSolder, F.Cu at (107.6, 50.4)
- added C12: 10nF, Capacitor_SMD:C_0805_2012Metric_Pad1.15x1.40mm_HandSolder, F.Cu at (102.8, 56.3)
- added C13: 1uF, Capacitor_SMD:C_0805_2012Metric_Pad1.15x1.40mm_HandSolder, F.Cu at (107.6, 53.4)
- added C7: 100nF, Capacitor_SMD:C_0805_2012Metric_Pad1.15x1.40mm_HandSolder, F.Cu at (102.8, 47.5)
- added C8: 100nF, Capacitor_SMD:C_0805_2012Metric_Pad1.15x1.40mm_HandSolder, F.Cu at (102.8, 50.4)
- added C9: 100nF, Capacitor_SMD:C_0805_2012Metric_Pad1.15x1.40mm_HandSolder, F.Cu at (107.6, 47.5)
- added U1: STM32F303CCT7, Package_QFP:LQFP-48_7x7mm_P0.5mm, F.Cu at (90.1, 51.1)
- REG2: value MIC2876-5.5YMT-TR -> MIC2876-5.0YMT-T5
Connections:
- BTN1 pad 1: BTN -> (no net)
- M1 pad 1: INDEX -> (no net)
- M2 pad 1: MIDDLE -> (no net)
- M3 pad 1: RING -> (no net)
- M4 pad 1: PINKY -> (no net)
- M5 pad 1: THUMB -> (no net)
- R7 pad 2: NEO -> (no net)
Routing:
- net (no net): track 0.00 -> 217.4 mm
- net RING: track 43.2 -> 0.00 mm
- net PINKY: track 39.2 -> 0.00 mm
- net INDEX: track 38.5 -> 0.00 mm
- net MIDDLE: track 33.2 -> 0.00 mm
- net THUMB: track 28.0 -> 0.00 mm
- net BTN: track 21.4 -> 0.00 mm
- net NEO: track 14.1 -> 0.00 mm
