File: v1.3/circuitdraft.brd (EAGLE design)
At the start: 31.2 x 35.4 mm, 25 parts, among them Y1 CY16BPS

Commit message: Started ahmad's changes
Routing:
- net GND: track 2.01 -> 0.00 mm
- net VBUS: track 26.9 -> 28.5 mm, vias 3 -> 2
- net BIGPOWER: track 42.5 -> 43.7 mm
- net STS: track 13.7 -> 14.3 mm
- net SIGNAL1: vias 2 -> 1
Changed lines of the file:
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@@
 <?xml version="1.0" encoding="utf-8"?>
 <!DOCTYPE eagle SYSTEM "eagle.dtd">
-<eagle version="9.5.1">
+<eagle version="9.5.2">
 <drawing>
 <settings>
@@
 <wire x1="35.052" y1="19.6596" x2="35.052" y2="17.2974" width="0.1524" layer="1"/>
 <wire x1="30.861" y1="23.8506" x2="35.052" y2="19.6596" width="0.1524" layer="16"/>
-<wire x1="30.861" y1="25.6032" x2="30.861" y2="23.8506" width="0.1524" layer="16"/>
-<wire x1="29.1084" y1="27.3558" x2="30.861" y2="25.6032" width="0.1524" layer="1"/>
-<wire x1="29.1084" y1="28.3464" x2="29.1084" y2="27.3558" width="0.1524" layer="1"/>
 <wire x1="28.7274" y1="12.7254" x2="28.72" y2="12.66" width="0.1524" layer="1"/>
-<wire x1="29.1084" y1="28.3464" x2="29.06" y2="28.4" width="0.1524" layer="1"/>
 <via x="35.052" y="19.6596" extent="1-16" drill="0.254"/>
-<via x="30.861" y="25.6032" extent="1-16" drill="0.254"/>
+<wire x1="29.06" y1="28.4" x2="29.06" y2="26.44" width="0.1524" layer="16"/>
+<wire x1="30.861" y1="24.639" x2="30.861" y2="23.8506" width="0.1524" layer="16"/>
+<wire x1="29.06" y1="26.44" x2="30.861" y2="24.639" width="0.1524" layer="16"/>
 </signal>
 <signal name="SIGNAL2">
@@
 <wire x1="15.5" y1="22.05" x2="15.5" y2="21.3" width="0.1524" layer="1"/>
 <via x="15.5" y="21.3" extent="1-16" drill="0.35"/>
-<via x="20.9" y="17.7" extent="1-16" drill="0.35"/>
 <wire x1="15.5" y1="21.3" x2="18.0394" y2="18.7606" width="0.1524" layer="16"/>
 <wire x1="18.0394" y1="18.7606" x2="18.572325" y2="18.7606" width="0.1524" layer="16"/>
-<wire x1="19.632925" y1="17.7" x2="20.9" y2="17.7" width="0.1524" layer="16"/>
-<wire x1="18.572325" y1="18.7606" x2="19.632925" y2="17.7" width="0.1524" layer="16"/>
-<wire x1="20.9" y1="17.7" x2="22.08" y2="17.7" width="0.1524" layer="1"/>
 <wire x1="22.08" y1="17.7" x2="22.12" y2="17.66" width="0.1524" layer="1"/>
+<wire x1="19.732925" y1="17.6" x2="23.6" y2="17.6" width="0.1524" layer="16"/>
+<wire x1="18.572325" y1="18.7606" x2="19.732925" y2="17.6" width="0.1524" layer="16"/>
 </signal>
 <signal name="MISO">
@@
 <contactref element="BOOSTCONVERTER" pad="2"/>
 <contactref element="BOOSTCONVERTER" pad="4"/>
-<wire x1="16.65" y1="29.4" x2="16.65" y2="30.05" width="0.1524" layer="1"/>
-<wire x1="16.65" y1="30.05" x2="16.9" y2="30.3" width="0.1524" layer="1"/>
 <contactref element="BOOSTCONVERTER" pad="7"/>
-<via x="15.1" y="32.5" extent="1-16" drill="0.35"/>
+<via x="14.7" y="32.7" extent="1-16" drill="0.35"/>
 <via x="15.1" y="29.2" extent="1-16" drill="0.35"/>
 <via x="18.9" y="30" extent="1-16" drill="0.35"/>
-<wire x1="16.65" y1="31.2" x2="16.7436" y2="31.1064" width="0.254" layer="1"/>
-<wire x1="16.9" y1="30.75486875" x2="16.9" y2="30.3" width="0.254" layer="1"/>
-<wire x1="16.7436" y1="31.1064" x2="16.7436" y2="30.91126875" width="0.254" layer="1"/>
-<wire x1="16.7436" y1="30.91126875" x2="16.9" y2="30.75486875" width="0.254" layer="1"/>
 <via x="24" y="19.3" extent="1-16" drill="0.35"/>
+<wire x1="16.9" y1="30.3" x2="16.65" y2="31.2" width="0" layer="19" extent="1-1"/>
 </signal>
 <signal name="INTERRUPT">
@@
 <wire x1="14" y1="17.77" x2="14" y2="25.4" width="1" layer="16"/>
 <wire x1="14" y1="25.4" x2="14.9" y2="26.3" width="1" layer="16"/>
-<via x="14.9" y="26.3" extent="1-16" drill="0.35"/>
+<via x="14.9" y="26.3" extent="1-16" drill="0.7" diameter="1"/>
 <wire x1="14.9" y1="26.3" x2="16.538" y2="26.3" width="1" layer="1"/>
 <contactref element="BOOSTCONVERTER" pad="3"/>
@@
 <wire x1="31.3406" y1="33.613525" x2="31.3406" y2="31.827675" width="0.1524" layer="16"/>
 <wire x1="31.3406" y1="31.827675" x2="30.760325" y2="31.2474" width="0.1524" layer="16"/>
-<wire x1="26.9306" y1="27.427675" x2="26.4" y2="26.897075" width="0.1524" layer="16"/>
-<wire x1="26.4" y1="26.897075" x2="26.4" y2="26.1" width="0.1524" layer="16"/>
+<wire x1="27.5306" y1="27.527675" x2="26.4" y2="26.397075" width="0.1524" layer="16"/>
+<wire x1="26.4" y1="26.397075" x2="26.4" y2="26.1" width="0.1524" layer="16"/>
 <wire x1="30.760325" y1="31.2474" x2="29.744475" y2="31.2474" width="0.1524" layer="16"/>
-<wire x1="29.744475" y1="31.2474" x2="26.9306" y2="28.433525" width="0.1524" layer="16"/>
-<wire x1="26.9306" y1="28.433525" x2="26.9306" y2="27.427675" width="0.1524" layer="16"/>
+<wire x1="29.744475" y1="31.2474" x2="27.5306" y2="29.033525" width="0.1524" layer="16"/>
+<wire x1="27.5306" y1="29.033525" x2="27.5306" y2="27.527675" width="0.1524" layer="16"/>
 <wire x1="26.4" y1="26.1" x2="26.4" y2="24.4188" width="0.1524" layer="1"/>
 <wire x1="26.4" y1="24.4188" x2="26.289" y2="24.3078" width="0.1524" layer="1"/>
@@
 <wire x1="25.5" y1="30.8236" x2="25.5" y2="34.675" width="1" layer="1"/>
 <wire x1="25.5" y1="34.675" x2="25.275" y2="34.9" width="1" layer="1"/>
-<wire x1="16.15" y1="31.2" x2="15.6" y2="31.75" width="0.4064" layer="1"/>
-<wire x1="15.6" y1="31.75" x2="15.6" y2="31.8" width="0.508" layer="1"/>
-<via x="15.6" y="31.8" extent="1-16" drill="0.35"/>
-<wire x1="15.6" y1="31.8" x2="16.5" y2="32.7" width="0.508" layer="16"/>
+<wire x1="16.15" y1="31.2" x2="15.2" y2="31.2" width="0.4064" layer="1"/>
+<wire x1="15.2" y1="31.9" x2="15.3" y2="32" width="0.508" layer="1"/>
+<wire x1="15.2" y1="31.9" x2="15.2" y2="31.2" width="0.508" layer="1"/>
+<via x="15.3" y="32" extent="1-16" drill="0.35"/>
+<wire x1="15.3" y1="32" x2="16" y2="32.7" width="0.508" layer="16"/>
 <via x="18.7" y="31.2" extent="1-16" drill="0.35"/>
 <wire x1="17.8584" y1="32.19343125" x2="17.8584" y2="32.0416" width="0.508" layer="16"/>
@@
 <wire x1="18.7" y1="31.2" x2="20.45" y2="31.2" width="0.508" layer="1"/>
 <wire x1="20.45" y1="31.2" x2="20.475" y2="31.225" width="0.508" layer="1"/>
-<wire x1="16.5" y1="32.7" x2="17.35183125" y2="32.7" width="0.508" layer="16"/>
+<wire x1="16" y1="32.7" x2="17.35183125" y2="32.7" width="0.508" layer="16"/>
 <wire x1="17.65" y1="31.2" x2="18.7" y2="31.2" width="0.4064" layer="1"/>
 </signal>
@@
 <contactref element="CHARGER" pad="1"/>
 <contactref element="U$1" pad="40"/>
-<wire x1="26.6646875" y1="23.2814" x2="27.12" y2="23.7367125" width="0.1524" layer="1"/>
-<wire x1="27.12" y1="23.7367125" x2="27.12" y2="24.26" width="0.1524" layer="1"/>
-<wire x1="22" y1="23.2814" x2="22.5" y2="23.2814" width="0.1524" layer="1"/>
-<wire x1="22.5" y1="23.2814" x2="26.6646875" y2="23.2814" width="0.1524" layer="1"/>
-<wire x1="21.0314" y1="23.2814" x2="22" y2="23.2814" width="0.1524" layer="1"/>
+<wire x1="26.8646875" y1="22.9814" x2="27.12" y2="23.2367125" width="0.1524" layer="1"/>
+<wire x1="27.12" y1="23.2367125" x2="27.12" y2="24.26" width="0.1524" layer="1"/>
+<wire x1="26.8646875" y1="22.9814" x2="22.8" y2="22.9814" width="0.1524" layer="1"/>
+<wire x1="22.5" y1="23.2814" x2="22.8" y2="22.9814" width="0.1524" layer="1"/>
+<wire x1="21.0314" y1="23.2814" x2="22.5" y2="23.2814" width="0.1524" layer="1"/>
 <wire x1="17.3053125" y1="20.6964" x2="17.1714" y2="20.8303125" width="0.1524" layer="1"/>
 <wire x1="18" y1="20.25" x2="17.5536" y2="20.6964" width="0.1524" layer="1"/>

Commit message: Jacks changes
Parts:
- added C5: (no value), 3DPC:C0603
- moved USB 22.5 mm to (15.5, 12.6), turned to 0 degrees
- moved BAT 3.22 mm to (14.2, 16.9)
- moved PWRSW 3.01 mm to (11.0, 16.8)
- moved RPROG 0.45 mm to (13.0, 21.6)
- moved CIN 0.40 mm to (14.0, 24.5)
- moved CHARGER 0.20 mm to (16.9, 21.2)
Connections:
- net VBUS: no longer U$1.7
Routing:
- net VBUS: track 28.5 -> 13.3 mm, vias 2 -> 1
- net N$5: track 0.03 -> 12.6 mm
- net N$6: track 0.01 -> 12.2 mm
- net POWER: track 46.4 -> 49.2 mm
- net BATCHARGE: track 13.1 -> 15.8 mm
- net SCK: track 13.5 -> 11.6 mm
- net INTERRUPT: track 23.6 -> 22.2 mm
- net MOSI: track 13.3 -> 14.7 mm
- net GND: track 0.00 -> 1.00 mm, vias 15 -> 14
- net N$4: track 2.24 -> 2.79 mm
- net VBAT: track 42.1 -> 41.5 mm, vias 5 -> 3
Other:
- board size 31.2 x 35.4 mm -> 49.3 x 49.3 mm
