File: v1.3/circuitdraft.sch (EAGLE design)
At the start: 25 parts, among them Y1 CY16BPS

Commit message: Jacks changes
Parts:
- added C5: (no value), 3DPC:C-USC0603
Connections:
- net VBUS: no longer U$1.VBUS
Changed lines of the file:
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@@
 <?xml version="1.0" encoding="utf-8"?>
 <!DOCTYPE eagle SYSTEM "eagle.dtd">
-<eagle version="9.5.1">
+<eagle version="9.5.2">
 <drawing>
 <settings>
@@
 <part name="AGND2" library="supply1" library_urn="urn:adsk.eagle:library:371" deviceset="GND" device=""/>
 <part name="L2" library="inductor-neosid" library_urn="urn:adsk.eagle:library:241" deviceset="SD75" device="" package3d_urn="urn:adsk.eagle:package:14650/1" value="1 μH"/>
+<part name="C5" library="3DPC" deviceset="C-US" device="C0603" package3d_urn="urn:adsk.eagle:package:23616/2"/>
 </parts>
 <sheets>
@@
 <attribute name="VALUE" x="74.93" y="62.484" size="1.778" layer="96"/>
 </instance>
+<instance part="C5" gate="G$1" x="27.94" y="213.36" smashed="yes">
+<attribute name="NAME" x="28.956" y="213.995" size="1.778" layer="95"/>
+<attribute name="VALUE" x="28.956" y="209.169" size="1.778" layer="96"/>
+</instance>
 </instances>
 <busses>
@@
 </segment>
 <segment>
-<pinref part="U$1" gate="G$1" pin="VBUS"/>
-<wire x1="137.16" y1="124.46" x2="134.62" y2="124.46" width="0.1524" layer="91"/>
-<label x="134.62" y="124.46" size="1.778" layer="95" rot="R180" xref="yes"/>
-</segment>
-<segment>
