File: v2.1/PCB/Hand v2.1.kicad_pcb (KiCad board)
At the start: 2 copper layers, 39 x 58 mm, 41 parts, among them J1 Conn_ARM_JTAG_SWD_10, M1 Index_Servo, M2 Middle_Servo, M3 Ring_Servo, M4 Pinky_Servo, M5 Thumb_Servo, SW1 Power_Switch, U1 STM32F303CCT7

Commit message: enabled regulators and removed unneeded part
Parts:
- removed R4: 1Mohm, Resistor_SMD:R_0805_2012Metric_Pad1.15x1.40mm_HandSolder
- C4: value 4.7uF 10V -> 4.7uF 10V X7R
- C6: value 22uF 10V -> 100uF 10V X7R
- L1: value 1uH 3A -> 1.5uH 3A
Connections:
- REG1 pad 3: (no net) -> +BATT
- REG2 pad 6: (no net) -> +BATT
- REG2 pad 7: Net-(R4-Pad2) -> GND
Routing:
- net +BATT: track 42.2 -> 47.0 mm
- net Net-(R4-Pad2): track 2.68 -> 0.00 mm
- net GND: track 63.0 -> 64.1 mm, vias 6 -> 7

Commit message: updated name of battery to be clearer
Parts:
- renumbered BT1 to BATT1
