File: v2.1/PCB/Hand v2.1.sch (KiCad schematic (older format))
At the start: 41 parts, among them J1 Conn_ARM_JTAG_SWD_10, M1 Index_Servo, M2 Middle_Servo, M3 Ring_Servo, M4 Pinky_Servo, M5 Thumb_Servo, SW1 Power_Switch, U1 STM32F303CCT7

Commit message: rename 2.0 to 2.1 for chip change
Parts:
- MYO1: symbol Hand-v2.0-Parts:MyoWare -> Hand-v2.1-rescue:MyoWare-Hand-v2.0-Parts-Hand-v2.1-rescue
- REG2: symbol Hand-v2.0-Parts:MIC2876-5.5YMT-TR -> Hand-v2.1-rescue:MIC2876-5.5YMT-TR-Hand-v2.0-Parts-Hand-v2.1-rescue
Changed lines of the file:
@@
 EESchema Schematic File Version 4
-LIBS:Hand v2.0-cache
+LIBS:Hand v2.1-cache
 EELAYER 30 0
 EELAYER END
@@
 $EndComp
 $Comp
-L Hand-v2.0-Parts:MyoWare MYO1
+L Hand-v2.1-rescue:MyoWare-Hand-v2.0-Parts-Hand-v2.1-rescue MYO1
 U 1 1 5E217809
 P 8550 4400
@@
 $EndComp
 $Comp
-L Hand-v2.0-Parts:MIC2876-5.5YMT-TR REG2
+L Hand-v2.1-rescue:MIC2876-5.5YMT-TR-Hand-v2.0-Parts-Hand-v2.1-rescue REG2
 U 1 1 5E2A2729
 P 4950 6450

Commit message: finished adding STM32F303VCT6
Connections:
- wire segments 105 -> 104
Changed lines of the file:
@@
 Text GLabel 9750 800  2    50   Input ~ 0
 MYOSIG
-Text GLabel 3800 2700 2    50   Input ~ 0
+Text GLabel 2750 3050 2    50   Input ~ 0
 NORMVBAT
 Text GLabel 7750 850  0    50   Input ~ 0
@@
 Wire Wire Line
 	7700 2950 7850 2950
-Text GLabel 3800 2500 2    50   Input ~ 0
+Text GLabel 2750 2950 2    50   Input ~ 0
 NORMMYOSIG
 Text GLabel 8250 4500 0    50   Input ~ 0
@@
 Text GLabel 8100 3700 0    50   Input ~ 0
 BTN
-Text GLabel 4050 3800 3    50   Input ~ 0
+Text GLabel 2750 3350 2    50   Input ~ 0
 BTN
 Wire Wire Line
-	4050 3500 4050 3800
-Wire Wire Line
-	4050 3500 4200 3500
-Wire Wire Line
 	8100 3700 8200 3700
-Text GLabel 3800 2600 2    50   Input ~ 0
+Text GLabel 2750 3150 2    50   Input ~ 0
 THUMB
 Wire Wire Line
-	3650 2500 3800 2500
-Wire Wire Line
-	3650 2600 3800 2600
-Wire Wire Line
-	3650 2700 3800 2700
-Text GLabel 3800 2800 2    50   Input ~ 0
+	2600 2950 2750 2950
+Wire Wire Line
+	2600 3150 2750 3150
+Wire Wire Line
+	2600 3050 2750 3050
+Text GLabel 2750 2550 2    50   Input ~ 0
 INDEX
-Text GLabel 3800 2900 2    50   Input ~ 0
+Text GLabel 2750 2650 2    50   Input ~ 0
 MIDDLE
-Text GLabel 3800 3000 2    50   Input ~ 0
+Text GLabel 2750 2750 2    50   Input ~ 0
 RING
-Text GLabel 3800 3100 2    50   Input ~ 0
+Text GLabel 2750 2850 2    50   Input ~ 0
 PINKY
 Wire Wire Line
-	3650 2800 3800 2800
-Wire Wire Line
-	3650 2900 3800 2900
-Wire Wire Line
-	3650 3000 3800 3000
-Wire Wire Line
-	3650 3100 3800 3100
-Text GLabel 4200 3800 3    50   Input ~ 0
+	2600 2550 2750 2550
+Wire Wire Line
+	2600 2650 2750 2650
+Wire Wire Line
+	2600 2750 2750 2750
+Wire Wire Line
+	2600 2850 2750 2850
+Text GLabel 2750 3250 2    50   Input ~ 0
 NEO
-Wire Wire Line
-	4200 3600 4200 3800
 $Comp
 L Device:R_US R8
@@
 Wire Wire Line
 	5600 1550 5050 1550
+Wire Wire Line
+	2750 3250 2600 3250
+Wire Wire Line
+	2750 3350 2600 3350
 $EndSCHEMATC

Commit message: connected unused IO pins on MCU to ground
Connections:
- net GND: now also U1.18 (PB0), U1.19 (PB1), U1.2 (PC13), U1.20 (PB2), U1.21 (PB10), U1.22 (PB11), U1.25 (PB12), U1.26 (PB13), U1.27 (PB14), U1.28 (PB15), U1.3 (PC14), U1.30 (PA9), U1.31 (PA10), U1.32 (PA11), U1.33 (PA12), U1.38 (PA15), U1.39 (PB3), U1.4 (PC15), U1.40 (PB4), U1.41 (PB5), U1.42 (PB6), U1.43 (PB7), U1.44 (BOOT0), U1.45 (PB8), U1.46 (PB9), U1.5 (PF0), U1.6 (PF1)
Changed lines of the file:
@@
 Wire Wire Line
 	2750 3350 2600 3350
+Wire Wire Line
+	1300 1650 1300 1850
+Wire Wire Line
+	1300 4250 1800 4250
+Connection ~ 1300 1850
+Wire Wire Line
+	1300 1850 1300 1950
+Connection ~ 1300 1950
+Wire Wire Line
+	1300 1950 1300 2150
+Connection ~ 1300 2150
+Wire Wire Line
+	1300 2150 1300 2250
+Connection ~ 1300 2250
+Wire Wire Line
+	1300 2250 1300 2350
+Connection ~ 1300 2350
+Wire Wire Line
+	1300 2350 1300 2550
+Connection ~ 1300 2550
+Wire Wire Line
+	1300 2550 1300 2650
+Connection ~ 1300 2650
+Wire Wire Line
+	1300 2650 1300 2750
+Connection ~ 1300 2750
+Wire Wire Line
+	1300 2750 1300 2850
+Connection ~ 1300 2850
+Wire Wire Line
+	1300 2850 1300 2950
+Connection ~ 1300 2950
+Wire Wire Line
+	1300 2950 1300 3050
+Connection ~ 1300 3050
+Wire Wire Line
+	1300 3050 1300 3150
+Connection ~ 1300 3150
+Wire Wire Line
+	1300 3150 1300 3250
+Connection ~ 1300 3250
+Wire Wire Line
+	1300 3250 1300 3350
+Connection ~ 1300 3350
+Wire Wire Line
+	1300 3350 1300 3450
+Connection ~ 1300 3450
+Wire Wire Line
+	1300 3450 1300 3550
+Connection ~ 1300 3550
+Wire Wire Line
+	1300 3550 1300 3650
+Connection ~ 1300 3650
+Wire Wire Line
+	1300 3650 1300 3750
+Connection ~ 1300 3750
+Wire Wire Line
+	1300 3750 1300 3850
+Connection ~ 1300 3850
+Wire Wire Line
+	1300 3850 1300 3950
+Connection ~ 1300 3950
+Wire Wire Line
+	1300 3950 1300 4050
+Connection ~ 1300 4050
+Wire Wire Line
+	1300 4050 1300 4250
+Connection ~ 1800 4250
+Wire Wire Line
+	2600 3450 2700 3450
+Wire Wire Line
+	2700 3450 2700 3550
+Wire Wire Line
+	2700 4250 2400 4250
+Connection ~ 2400 4250
+Wire Wire Line
+	2600 3550 2700 3550
+Connection ~ 2700 3550
+Wire Wire Line
+	2700 3550 2700 3650
+Wire Wire Line
+	2600 3650 2700 3650
+Connection ~ 2700 3650
+Wire Wire Line
+	2700 3650 2700 3750
+Wire Wire Line
+	2600 3750 2700 3750
+Connection ~ 2700 3750
+Wire Wire Line
+	2700 3750 2700 4050
+Wire Wire Line
+	2600 4050 2700 4050
+Connection ~ 2700 4050
+Wire Wire Line
+	2700 4050 2700 4250
 $EndSCHEMATC

Commit message: enabled regulators and removed unneeded part
Parts:
- removed R4: 1Mohm, Resistor_SMD:R_0805_2012Metric_Pad1.15x1.40mm_HandSolder, symbol Device:R_US
- C4: value 4.7uF 10V -> 4.7uF 10V X7R
- C6: value 22uF 10V -> 100uF 10V X7R
- L1: value 1uH 3A -> 1.5uH 3A
Connections:
- net +BATT: now also REG1.3 (EN), REG2.6 (EN)
- net GND: now also REG2.7 (/PG)
Changed lines of the file:
@@
 EESchema Schematic File Version 4
-LIBS:Hand v2.1-cache
 EELAYER 30 0
 EELAYER END
@@
 P 4050 6700
 F 0 "L1" H 4102 6746 50  0000 L CNN
-F 1 "1uH 3A" H 4102 6655 50  0000 L CNN
+F 1 "1.5uH 3A" H 4102 6655 50  0000 L CNN
 F 2 "Inductor_SMD:L_1210_3225Metric_Pad1.42x2.65mm_HandSolder" H 4050 6700 50  0001 C CNN
 F 3 "~" H 4050 6700 50  0001 C CNN
@@
 P 4050 7000
 F 0 "C4" H 4165 7046 50  0000 L CNN
-F 1 "4.7uF 10V" H 4165 6955 50  0000 L CNN
+F 1 "4.7uF 10V X7R" H 4165 6955 50  0000 L CNN
 F 2 "Capacitor_SMD:C_0805_2012Metric_Pad1.15x1.40mm_HandSolder" H 4088 6850 50  0001 C CNN
 F 3 "~" H 4050 7000 50  0001 C CNN
@@
 P 6300 6800
 F 0 "C6" H 6415 6846 50  0000 L CNN
-F 1 "22uF 10V" H 6415 6755 50  0000 L CNN
+F 1 "100uF 10V X7R" H 6415 6755 50  0000 L CNN
 F 2 "Capacitor_SMD:C_0805_2012Metric_Pad1.15x1.40mm_HandSolder" H 6338 6650 50  0001 C CNN
 F 3 "~" H 6300 6800 50  0001 C CNN
 	1    6300 6800
-	1    0    0    -1
-$EndComp
-$Comp
-L Device:R_US R4
-U 1 1 5E2AE730
-P 5850 6200
-F 0 "R4" H 5918 6246 50  0000 L CNN
-F 1 "1Mohm" H 5918 6155 50  0000 L CNN
-F 2 "Resistor_SMD:R_0805_2012Metric_Pad1.15x1.40mm_HandSolder" V 5890 6190 50  0001 C CNN
-F 3 "~" H 5850 6200 50  0001 C CNN
-	1    5850 6200
 	1    0    0    -1
 $EndComp
@@
 	1    0    0    -1
 $EndComp
-Wire Wire Line
-	3600 6850 4050 6850
 Connection ~ 4050 6850
 Wire Wire Line
@@
 Wire Wire Line
 	4700 6550 4050 6550
-$Comp
-L power:+BATT #PWR016
-U 1 1 5E2B9E39
-P 5850 6050
-F 0 "#PWR016" H 5850 5900 50  0001 C CNN
-F 1 "+BATT" H 5865 6223 50  0000 C CNN
-F 2 "" H 5850 6050 50  0001 C CNN
-F 3 "" H 5850 6050 50  0001 C CNN
-	1    5850 6050
-	1    0    0    -1
-$EndComp
 Wire Wire Line
 	5650 6750 5850 6750
-Wire Wire Line
-	5850 6750 5850 6350
 $Comp
 L power:+5V #PWR018
@@
 Wire Wire Line
 	2700 4050 2700 4250
+Wire Wire Line
+	3600 6850 3850 6850
+Wire Wire Line
+	5650 6850 5750 6850
+Wire Wire Line
+	5750 6850 5750 7400
+Wire Wire Line
+	5750 7400 3850 7400
+Wire Wire Line
+	3850 7400 3850 6850
+Connection ~ 3850 6850
+Wire Wire Line
+	3850 6850 4050 6850
+Wire Wire Line
+	5850 6750 5850 7150
+Wire Wire Line
+	5850 7150 5150 7150
+Connection ~ 5150 7150
+Wire Wire Line
+	5000 4750 5000 4550
+Connection ~ 5000 4550
 $EndSCHEMATC

Commit message: updated name of battery to be clearer
Parts:
- renumbered BT1 to BATT1
Changed lines of the file:
@@
 $EndComp
 $Comp
-L Device:Battery_Cell BT1
+L Device:Battery_Cell BATT1
 U 1 1 5E26E216
 P 10500 5450
-F 0 "BT1" H 10618 5546 50  0000 L CNN
+F 0 "BATT1" H 10618 5546 50  0000 L CNN
 F 1 "Battery_Cell" H 10618 5455 50  0000 L CNN
 F 2 "Connector_JST:JST_EH_S2B-EH_1x02_P2.50mm_Horizontal" V 10500 5510 50  0001 C CNN
