File: v3.0/hand v3.0/hand v3.0.sch (KiCad schematic (older format))
At the start: 15 parts

Commit message: motor and motor drivers configured
Parts:
- added C? (x8): 0.1uF, symbol Device:C
- added M? (x5): PQ12-P, symbol Hand~Parts:PQ12-P
- added U? (x4): DRV8838, Package_SON:WSON-8-1EP_2x2mm_P0.5mm_EP0.9x1.6mm, symbol Driver_Motor:DRV8838
Connections:
- net labels added: MOTOR_1_DIR, MOTOR_1_POS, MOTOR_1_PWM, MOTOR_2_DIR, MOTOR_2_POS, MOTOR_2_PWM, MOTOR_3_DIR, MOTOR_3_POS, MOTOR_3_PWM, MOTOR_4_DIR, MOTOR_4_POS, MOTOR_4_PWM, MOTOR_5_DIR, MOTOR_5_POS, MOTOR_5_PWM
- wire segments 24 -> 111
Other:
- moved on the sheet: BT?, C?, D?, R?, SW?, U?
